File: soup-soup-soup-sahur.kicad_pcb (KiCad board)
At the start: 2 copper layers, 70 x 100 mm, 13 parts, among them J1 USB_C_Receptacle_USB2.0_14P, U1 NT3H2111W0FHKH

Commit message: triple s but better
Parts:
- removed the G*** at (102.9, 81.9)
- moved J1 49.5 mm to (122.8, 85.2), turned to 90 degrees
- moved R1 42.2 mm to (110.1, 85.7)
- moved R2 41.3 mm to (110.1, 84.2)
- moved ANT1 0.10 mm to (103.8, 70.1)
Routing:
- net /explodey thing: track 69.4 -> 35.8 mm
- net GND: track 5.73 -> 11.3 mm, vias 54 -> 21
- net Net-(J1-CC1): track 11.2 -> 9.95 mm, vias 0 -> 2
- net Net-(J1-CC2): track 9.85 -> 9.91 mm, vias 0 -> 2
Other:
- board size 70 x 100 mm -> 59.1 x 91.7 mm
- board text added: "5v power go 2v cap cap go kaboom"
- board text added: "github: @0x62b codeberg: @0x62b hc slack: @0x62 web: https://0x62.dev mail: benjamin@0x62.dev"
- board text added: "soup soup soup sahur (triple s)"
- board text removed: "github: @0x62b codeberg: @0x62b hc slack: @0x62 signal: benjamin.492 web: https://0x62.dev mail: benjamin@0x62.dev"

Commit message: idfk
Routing:
- net /explodey thing: track 35.8 -> 34.8 mm
Changed lines of the file:
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@@
-	)
-	(segment
-		(start 106.8 69.7075)
-		(end 107.9075 68.6)
-		(width 0.4)
-		(layer "F.Cu")
-		(net "/explodey thing")
 	)
 	(segment
 		(start 119.88 83.086016)
 		(end 119.88 87.22383)
-		(width 0.4)
-		(layer "F.Cu")
-		(net "/explodey thing")
-	)
-	(segment
-		(start 107.9075 68.6)
-		(end 107.9075 64.9)
 		(width 0.4)
 		(layer "F.Cu")
@@
 	)
 	(segment
-		(start 106.8 80.7)
-		(end 106.8 69.7075)
+		(start 107.9075 81.8075)
+		(end 107.9075 64.9)
 		(width 0.4)
 		(layer "F.Cu")
@@
 	)
 	(via
-		(at 106.8 80.7)
+		(at 107.9075 81.8075)
 		(size 0.8)
 		(drill 0.4)
@@
 	)
 	(segment
-		(start 106.8 80.7)
+		(start 107.9075 81.8075)
 		(end 108.5 82.4)
 		(width 0.4)
